Commit message: Made most of the changes requested for pull request. Still need to move blending and intrinsic cal demo to different repository

File: industrial_extrinsic_cal/urdf/calibration_transform_macro.xacro (robot description, xacro)
@@ -19,5 +19,5 @@
                     <origin xyz="0 0 0" rpy="0 0 0" />
                     <axis xyz="1 0 0" rpy="0 0 0" />
-	     <limit lower="-1.0" upper="1.0" effort="30" velocity="0.0508"/>
+	     <!--limit lower="-1.0" upper="1.0" effort="30" velocity="0.0508"/-->
 	</joint>
                <joint name="${child_link}_y_joint" type="prismatic">
@@ -26,5 +26,5 @@
                     <origin xyz="0 0 0" rpy="0 0 0" />
                     <axis xyz="0 1 0" rpy="0 0 0"/>
-	     <limit lower="-1.0" upper="1.0" effort="30" velocity="0.0508"/>
+	     <!--limit lower="-1.0" upper="1.0" effort="30" velocity="0.0508"/-->
 	</joint>
                <joint name="${child_link}_z_joint" type="prismatic">
@@ -33,5 +33,5 @@
                     <origin xyz="0 0 0" rpy="0 0 0" />
                     <axis xyz="0 0 1" rpy="0 0 0"/>
-	     <limit lower="-1.0" upper="1.0" effort="30" velocity="0.0508"/>
+	     <!--limit lower="-1.0" upper="1.0" effort="30" velocity="0.0508"/-->
 	</joint>
                <joint name="${child_link}_yaw_joint" type="revolute">
@@ -39,5 +39,5 @@
 	     <child  link="${child_link}_yaw" />
                     <origin xyz="0 0 0" rpy="0 0 0" />
-	     <limit lower="-3.1415" upper="3.1415" effort="2" velocity="10"/>
+	     <!--limit lower="-3.1415" upper="3.1415" effort="2" velocity="10"/-->
                     <axis xyz="0 0 1" />
 	</joint>
@@ -46,5 +46,5 @@
 	     <child  link="${child_link}_pitch"/>
                     <origin xyz="0 0 0" rpy="0 0 0" />
-	     <limit lower="-3.1415" upper="3.1415" effort="2" velocity="10"/>
+	     <!--limit lower="-3.1415" upper="3.1415" effort="2" velocity="10"/-->
                     <axis xyz="0 1 0" />
 	</joint>
@@ -53,5 +53,5 @@
 	     <child  link="${child_link}" />
                     <origin xyz="0 0 0" rpy="0 0 0" />
-	     <limit lower="-3.1415" upper="3.1415" effort="2" velocity="10"/>
+	     <!--limit lower="-3.1415" upper="3.1415" effort="2" velocity="10"/-->
                     <axis xyz="1 0 0" />
 	</joint>

Commit message: CMakeLists change for handleing Eigen calibration_job_definition change to update to new yaml-cpp interface, plus removed an unused variable mutable_joint_state publisher updated to new yaml-cpp interface calibration_transform_macro reinstalled joint limits, don't know why these need to be there perhaps can remove in future

File: industrial_extrinsic_cal/urdf/calibration_transform_macro.xacro (robot description, xacro)
@@ -19,5 +19,5 @@
                     <origin xyz="0 0 0" rpy="0 0 0" />
                     <axis xyz="1 0 0" rpy="0 0 0" />
-	     <!--limit lower="-1.0" upper="1.0" effort="30" velocity="0.0508"/-->
+	     <limit lower="-1.0" upper="1.0" effort="30" velocity="0.0508"/>
 	</joint>
                <joint name="${child_link}_y_joint" type="prismatic">
@@ -26,5 +26,5 @@
                     <origin xyz="0 0 0" rpy="0 0 0" />
                     <axis xyz="0 1 0" rpy="0 0 0"/>
-	     <!--limit lower="-1.0" upper="1.0" effort="30" velocity="0.0508"/-->
+	     <limit lower="-1.0" upper="1.0" effort="30" velocity="0.0508"/>
 	</joint>
                <joint name="${child_link}_z_joint" type="prismatic">
@@ -33,5 +33,5 @@
                     <origin xyz="0 0 0" rpy="0 0 0" />
                     <axis xyz="0 0 1" rpy="0 0 0"/>
-	     <!--limit lower="-1.0" upper="1.0" effort="30" velocity="0.0508"/-->
+	     <limit lower="-1.0" upper="1.0" effort="30" velocity="0.0508"/>
 	</joint>
                <joint name="${child_link}_yaw_joint" type="revolute">
@@ -39,5 +39,5 @@
 	     <child  link="${child_link}_yaw" />
                     <origin xyz="0 0 0" rpy="0 0 0" />
-	     <!--limit lower="-3.1415" upper="3.1415" effort="2" velocity="10"/-->
+	     <limit lower="-3.1415" upper="3.1415" effort="2" velocity="10"/>
                     <axis xyz="0 0 1" />
 	</joint>
@@ -46,5 +46,5 @@
 	     <child  link="${child_link}_pitch"/>
                     <origin xyz="0 0 0" rpy="0 0 0" />
-	     <!--limit lower="-3.1415" upper="3.1415" effort="2" velocity="10"/-->
+	     <limit lower="-3.1415" upper="3.1415" effort="2" velocity="10"/>
                     <axis xyz="0 1 0" />
 	</joint>
@@ -53,5 +53,5 @@
 	     <child  link="${child_link}" />
                     <origin xyz="0 0 0" rpy="0 0 0" />
-	     <!--limit lower="-3.1415" upper="3.1415" effort="2" velocity="10"/-->
+	     <limit lower="-3.1415" upper="3.1415" effort="2" velocity="10"/>
                     <axis xyz="1 0 0" />
 	</joint>

Commit message: added manual calt adjuster added params to control gen of post proc data removed parsing of scene_id to make concatenation of caljobs easier removed unused parameters for saving transform results from parser/caljob added params to control overwrite of mutable joint file removed superflous header of mutable.yaml file fixed yet another error in sorting for modified circle grid finder changed limits on the calibrateable transform xacro to hide moveit bug

File: industrial_extrinsic_cal/urdf/calibration_transform_macro.xacro (robot description, xacro)
@@ -39,5 +39,5 @@
 	     <child  link="${child_link}_yaw" />
                     <origin xyz="0 0 0" rpy="0 0 0" />
-	     <limit lower="-3.1415" upper="3.1415" effort="2" velocity="10"/>
+	     <limit lower="-6.2832" upper="6.2832" effort="2" velocity="10"/>
                     <axis xyz="0 0 1" />
 	</joint>
@@ -46,5 +46,5 @@
 	     <child  link="${child_link}_pitch"/>
                     <origin xyz="0 0 0" rpy="0 0 0" />
-	     <limit lower="-3.1415" upper="3.1415" effort="2" velocity="10"/>
+	     <limit lower="-6.2832" upper="6.2832" effort="2" velocity="10"/>
                     <axis xyz="0 1 0" />
 	</joint>
@@ -53,5 +53,5 @@
 	     <child  link="${child_link}" />
                     <origin xyz="0 0 0" rpy="0 0 0" />
-	     <limit lower="-3.1415" upper="3.1415" effort="2" velocity="10"/>
+	     <limit lower="-6.2832" upper="6.2832" effort="2" velocity="10"/>
                     <axis xyz="1 0 0" />
 	</joint>

Commit message: Fix indentation in calibration transform macro

File: industrial_extrinsic_cal/urdf/calibration_transform_macro.xacro (robot description, xacro)
@@ -1,59 +1,59 @@
 <?xml version="1.0" ?>
 <robot name="calibration_xform" xmlns:xacro="http://ros.org/wiki/xacro">
-      <xacro:macro name="calibration_definitions" params="child_link parent_link">
-    	<link name="${child_link}_x_trans">
-		<visual>
-			<origin rpy="0 0 0" xyz="0 0 0"/>
-			<geometry>
-				<sphere radius="0.0005"/>
-			</geometry>
-		</visual>
-                </link>
-          	<link name="${child_link}_y_trans"/>
-           	<link name="${child_link}_z_trans"/>
-           	<link name="${child_link}_pitch"/>
-           	<link name="${child_link}_yaw"/>
-               <joint name="${child_link}_x_joint" type="prismatic">
-                    <parent link="${parent_link}" />
-	     <child  link="${child_link}_x_trans" />
-                    <origin xyz="0 0 0" rpy="0 0 0" />
-                    <axis xyz="1 0 0" rpy="0 0 0" />
-	     <limit lower="-1.0" upper="1.0" effort="30" velocity="0.0508"/>
-	</joint>
-               <joint name="${child_link}_y_joint" type="prismatic">
-                    <parent link="${child_link}_x_trans" />
-	     <child  link="${child_link}_y_trans" />
-                    <origin xyz="0 0 0" rpy="0 0 0" />
-                    <axis xyz="0 1 0" rpy="0 0 0"/>
-	     <limit lower="-1.0" upper="1.0" effort="30" velocity="0.0508"/>
-	</joint>
-               <joint name="${child_link}_z_joint" type="prismatic">
-                    <parent link="${child_link}_y_trans" />
-	     <child  link="${child_link}_z_trans" />
-                    <origin xyz="0 0 0" rpy="0 0 0" />
-                    <axis xyz="0 0 1" rpy="0 0 0"/>
-	     <limit lower="-1.0" upper="1.0" effort="30" velocity="0.0508"/>
-	</joint>
-               <joint name="${child_link}_yaw_joint" type="revolute">
-                    <parent link="${child_link}_z_trans" />
-	     <child  link="${child_link}_yaw" />
-                    <origin xyz="0 0 0" rpy="0 0 0" />
-	     <limit lower="-6.2832" upper="6.2832" effort="2" velocity="10"/>
-                    <axis xyz="0 0 1" />
-	</joint>
-               <joint name="${child_link}_pitch_joint" type="revolute">
-                    <parent link="${child_link}_yaw" />
-	     <child  link="${child_link}_pitch"/>
-                    <origin xyz="0 0 0" rpy="0 0 0" />
-	     <limit lower="-6.2832" upper="6.2832" effort="2" velocity="10"/>
-                    <axis xyz="0 1 0" />
-	</joint>
-               <joint name="${child_link}_roll_joint" type="revolute">
-                    <parent link="${child_link}_pitch" />
-	     <child  link="${child_link}" />
-                    <origin xyz="0 0 0" rpy="0 0 0" />
-	     <limit lower="-6.2832" upper="6.2832" effort="2" velocity="10"/>
-                    <axis xyz="1 0 0" />
-	</joint>
-     </xacro:macro>
+  <xacro:macro name="calibration_definitions" params="child_link parent_link">
+    <link name="${child_link}_x_trans">
+      <visual>
+        <origin rpy="0 0 0" xyz="0 0 0"/>
+        <geometry>
+          <sphere radius="0.0005"/>
+        </geometry>
+      </visual>
+    </link>
+    <link name="${child_link}_y_trans"/>
+    <link name="${child_link}_z_trans"/>
+    <link name="${child_link}_pitch"/>
+    <link name="${child_link}_yaw"/>
+    <joint name="${child_link}_x_joint" type="prismatic">
+      <parent link="${parent_link}"/>
+      <child  link="${child_link}_x_trans"/>
+      <origin xyz="0 0 0" rpy="0 0 0"/>
+      <axis xyz="1 0 0" rpy="0 0 0"/>
+      <limit lower="-1.0" upper="1.0" effort="30" velocity="0.0508"/>
+    </joint>
+    <joint name="${child_link}_y_joint" type="prismatic">
+      <parent link="${child_link}_x_trans"/>
+      <child  link="${child_link}_y_trans"/>
+      <origin xyz="0 0 0" rpy="0 0 0"/>
+      <axis xyz="0 1 0" rpy="0 0 0"/>
+      <limit lower="-1.0" upper="1.0" effort="30" velocity="0.0508"/>
+    </joint>
+    <joint name="${child_link}_z_joint" type="prismatic">
+      <parent link="${child_link}_y_trans"/>
+      <child  link="${child_link}_z_trans"/>
+      <origin xyz="0 0 0" rpy="0 0 0"/>
+      <axis xyz="0 0 1" rpy="0 0 0"/>
+      <limit lower="-1.0" upper="1.0" effort="30" velocity="0.0508"/>
+    </joint>
+    <joint name="${child_link}_yaw_joint" type="revolute">
+      <parent link="${child_link}_z_trans"/>
+      <child  link="${child_link}_yaw"/>
+      <origin xyz="0 0 0" rpy="0 0 0"/>
+      <limit lower="-6.2832" upper="6.2832" effort="2" velocity="10"/>
+      <axis xyz="0 0 1"/>
+    </joint>
+    <joint name="${child_link}_pitch_joint" type="revolute">
+      <parent link="${child_link}_yaw"/>
+      <child  link="${child_link}_pitch"/>
+      <origin xyz="0 0 0" rpy="0 0 0"/>
+      <limit lower="-6.2832" upper="6.2832" effort="2" velocity="10"/>
+      <axis xyz="0 1 0"/>
+    </joint>
+    <joint name="${child_link}_roll_joint" type="revolute">
+      <parent link="${child_link}_pitch"/>
+      <child  link="${child_link}"/>
+      <origin xyz="0 0 0" rpy="0 0 0"/>
+      <limit lower="-6.2832" upper="6.2832" effort="2" velocity="10"/>
+      <axis xyz="1 0 0"/>
+    </joint>
+  </xacro:macro>
 </robot>
