Commit message: Target's now generate own points,    updated parser to use parameters for point autogen    updated calibration_job_def to auto-display targets as markers    added a node for displaying autogen targets Removed sleep from ros_robot_scene_trigger to speed motion, add back if robot shakes too much for calibration use Added camera info url parameter to the single_sensor.launch improved caljob_creator with new parameters Added a new node to caljob_creator package to store and execute a sequence of joint moves

File: industrial_extrinsic_cal/urdf/asus_sensor_cal_macro.xacro (robot description, xacro)
@@ -58,5 +58,5 @@
 		<parent link="${prefix}_frame"/>
 		<child link="${prefix}_ir_link"/>
-		<origin rpy="0 0 0" xyz="0 0 0"/>
+		<origin rpy="0 0 0" xyz="0 0.05 0"/>
 	</joint>
 	<joint name="${prefix}_ir_optical_frame_joint" type="fixed">
