Commit message: fixed rviz cal gui to include load and covariance buttons, wrist cal now calls start on first obs, other minor changes

File: industrial_extrinsic_cal/urdf/astra_cal_macro.xacro (robot description, xacro)
@@ -16,7 +16,7 @@
 	<link name="${prefix}_link">
 		<visual>
-			<origin rpy="0 0 0" xyz="0 0 -${astra_lengthD2}"/>
+			<origin rpy="0 0 0" xyz="0 -${astra_lengthD2} 0 "/>
 			<geometry>
-				<box size="${astra_width} ${astra_height} ${astra_length}"/>
+				<box size="${astra_width} ${astra_length} ${astra_height} "/>
 			</geometry>
 			<material name="${prefix}dark_silver"/>

Commit message: Change camera yaml file to astra and modify astra macro

File: industrial_extrinsic_cal/urdf/astra_cal_macro.xacro (robot description, xacro)
@@ -13,5 +13,5 @@
 	<!-- links: one for the optical frame and one for defining the link geometry -->
 	<link name="${prefix}"/>
-	<link name="${prefix}_optical_frame"/>
+        <!-- <link name="${prefix}_optical_frame"/>-->
 	<link name="${prefix}_link">
 		<visual>
@@ -39,9 +39,9 @@
 	</joint>
 	<!-- joint to attach the camera geometry to the optical frame -->
-	<joint name="${prefix}_optical_joint" type="fixed">
+        <!--<joint name="${prefix}_optical_joint" type="fixed">
 		<parent link="${prefix}"/>
 		<child link="${prefix}_link"/>
 		<origin rpy="0 0 0" xyz="0 0 0"/>
-	</joint>
+        </joint>-->
      </xacro:macro>
 </robot>
